File: Hardware/0. Project/ElectronSheriff.sch (EAGLE design)
At the start: 81 parts, among them CN1 MicroSD Card, CN2 DISPLAY-OLED-128X64-I2C, J5 CORTEX_DEBUGPTH, Q1 BC817, Q2 AO3400, Q3 AO3400, U1 ADG774, U2 MAX4239, U3 NRF52832, U4 GL823, U5 LM321MF, U6 ADG774, U7 MAX4239, Y1 32MHz, Y2 32.768kHz

Commit message: MCU pins assignment
Parts:
- removed BT1: CR2450, 1053:1053
- removed J5: CORTEX_DEBUGPTH, SparkFun-Connectors:CORTEX_DEBUGPTH
- removed L3: BLM15HB221SN1, inductors:BLM15HB221SN1
- removed R26: 220R (5%), rcl:R-EU_R0603
- added J2: CORTEX_DEBUGPTH, SparkFun-Connectors:CORTEX_DEBUGPTH
- added L2: 3.9nH, nrf52832-breakout-temp:INDUCTOR-0402-3.9NH
- added R11: 10k (5%), rcl:R-EU_R0603
- added U8: CR2450, 1053:1053
- C1: value 10pF -> 100 nF
- C10: value 15 pF -> 100nF
- C11: value DNP -> 100 nF
- C12: value 6 pF -> DNP
- C13: value 15 pF -> 100 pF
- C14: value 0.8 pF -> 100 nF
- C15, C19, C7: value 100 nF -> 100nF
- C16: value 1uF -> 6 pF
- C17: value 100nF -> DNP
- C18: value 100 nF -> 6 pF
- C2: value 10pF -> 100nF
- C21: value 4.7 uF -> 10pF
- C22: value 10uF -> 15 pF; device rcl:C-EUC0805 -> rcl:C-EUC0603
- C23: value 100nF -> 0.8 pF
- C24: value 100nF -> 15 pF
- C26: value 10uF -> 100 nF
- C27: value 100nF -> 10pF
- C29: value 100nF -> 1uF
- C4: value 100nF -> 100 nF
- C5: value DNP -> 10uF; device rcl:C-EUC0603 -> rcl:C-EUC0805
- C6: value 100 pF -> 10uF
- C8: value 100 nF -> 4.7 uF
- C9: value 6 pF -> 100nF
- CN1: value MicroSD Card -> DISPLAY-OLED-128X64-I2C; device Micro SD:MICROSD-PUSH-OUT -> diy-modules:DISPLAY-OLED-128X64-I2C
- CN2: value DISPLAY-OLED-128X64-I2C -> MicroSD Card; device diy-modules:DISPLAY-OLED-128X64-I2C -> Micro SD:MICROSD-PUSH-OUT
- L1: value 3.9nH -> BLM15HB221SN1; device nrf52832-breakout-temp:INDUCTOR-0402-3.9NH -> inductors:BLM15HB221SN1
- Q1: value BC817 -> AO3400; device transistor-npn:BC817-16LT1SMD -> AO3400:AO3400
- Q2: value AO3400 -> BC817; device AO3400:AO3400 -> transistor-npn:BC817-16LT1SMD
- R10: value 0.01R (0.1%) -> 4K7 (5%)
- R12: value 0R (5%) -> 0.01R (0.1%)
- R13, R20: value 10k (5%) -> 220R (5%)
- R14, R17: value 10k (5%) -> 22k (0.05%)
- R15, R18: value 10k (5%) -> 68k (0.05%)
- R16: value 10k (5%) -> 10k (0.05%)
- R19: value 4K7 (5%) -> 10k (0.05%)
- R21: value 22k (0.05%) -> 10k (5%)
- R22: value 680R (5%) -> 10k (5%)
- R23: value 1k (5%) -> 10k (5%)
- R24: value 68k (0.05%) -> 10k (5%)
- R25: value 10k (0.05%) -> 10k (5%)
- R4: value 22k (0.05%) -> 0R (5%)
- R5: value 68k (0.05%) -> 1k (5%)
- R6: value 10k (0.05%) -> 680R (5%)
- R7: value 220R (5%) -> 10k (0.05%)
- R8: value 10k (0.05%) -> 10R (0.05%)
- R9: value 10R (0.05%) -> 10k (5%)
- U1: value ADG774 -> LM321MF; device ADG774:ADG774 -> linear:LM321MF
- U2: value MAX4239 -> GL823; device MAX4239AUT+:MAX4239AUTT -> GL823:GL823(B)HG
- U4: value GL823 -> ADG774; device GL823:GL823(B)HG -> ADG774:ADG774
- U5: value LM321MF -> MAX4239; device linear:LM321MF -> MAX4239AUT+:MAX4239AUTT
- U6: value ADG774 -> MAX4239; device ADG774:ADG774 -> MAX4239AUT+:MAX4239AUTT
- U7: value MAX4239 -> ADG774; device MAX4239AUT+:MAX4239AUTT -> ADG774:ADG774
- X1: device con-ptr500:AK500/2-H -> con-berg:PN87520
- X2: device con-berg:PN87520 -> con-ptr500:AK500/2-H
Connections:
- net P26 renamed MCU_UART_TX
- net P27 renamed MCU_UART_RX
- removed net ADC_AMMETER_VOUT: R26.2
- removed net ADC_VGND: R12.2
- removed net BLE_ANT: C14.1, L1.2, U3.ANT
- removed net DISPLAY_I2C_SCL: CN2.SCL, R16.1
- removed net DISPLAY_I2C_SDA: CN2.SDA, R17.1
- removed net MCU_TDI: J5.NC/TDI
- removed net P07: U3.P0.07
- removed net P08: U3.P0.08
- new net MCU_ADC_AMMETER_VOUT: R20.2
- new net MCU_ADC_VGND: R4.2
- new net MCU_BLE_ANT: C23.1, L2.2, U3.ANT
- new net MCU_I2C_SCL: CN1.SCL, R22.1, U3.P0.07
- new net MCU_I2C_SDA: CN1.SDA, R24.1, U3.P0.08
- net !MCU_RESET!: now also J2.!RESET; no longer J5.!RESET
- net !MCU_SPI_CS!: now also U4.S4B; no longer U1.S4B
- net +5V: now also C1.1, C20.1, C26.1, C28.1, C29.1, C32.1, C9.1, CN1.VCC, CN2.4, J2.VCC, R11.2, R21.2, R22.2, R23.2, R24.2, R25.2, U1.V+, U4.VDD, U5.!SHDN, U5.VCC, U6.!SHDN, U6.VCC, U7.VDD, U8.3V; no longer BT1.3V, C15.1, C16.1, C17.1, C21.1, C23.1, C24.1, C3.1, CN1.4, CN2.VCC, J5.VCC, R13.2, R14.2, R15.2, R16.2, R17.2, R18.2, U1.VDD, U2.!SHDN, U2.VCC, U5.V+, U6.VDD, U7.!SHDN, U7.VCC
- net 0V: now also C1.2, C10.1, C15.1, C2.2, C26.2, C28.2, C29.2, C3.1, C32.2, C6.1, C7.1, CN1.GND, CN2.10, CN2.6, J2.GND@3, J2.GND@5, J2.GNDDTCT, Q2.E, R6.2, R9.2, U1.V-, U2.GPIO3, U2.GPIO6, U2.SCL, U2.SDA, U2.SD_WP, U2.TEST, U4.!EN!, U4.VSS, U5.GND, U6.GND, U7.!EN!, U7.VSS, U8.GND, X1.4; no longer BT1.GND, C10.2, C15.2, C21.2, C26.1, C27.1, C28.1, C29.1, C3.2, C32.1, C6.2, C7.2, CN1.10, CN1.6, CN2.GND, J5.GND@3, J5.GND@5, J5.GNDDTCT, Q1.E, R20.2, R22.2, U1.!EN!, U1.VSS, U4.GND, U4.GPIO3, U4.GPIO6, U4.SCL, U4.SDA, U4.SD_WP, U4.TEST, U5.V-, U6.!EN!, U6.VSS, U7.GND, X2.4
- net ADC_AMMETER: now also C21.1, R14.2, U5.OUT, U6.IN+; no longer C1.1, R4.2, U2.OUT, U7.IN+
- net ADC_AMMETER1: now also C27.1, R17.2, R20.1, U6.OUT; no longer C2.1, R21.2, R26.1, U7.OUT
- net CRYSTAL_XC1: now also C16.1; no longer C12.1
- net CRYSTAL_XC2: now also C18.1; no longer C9.1
- net CRYSTAL_XL1: now also C22.1; no longer C10.1
- net CRYSTAL_XL2: now also C24.1; no longer C13.1
- net MCU_SPI_CLK: now also U7.S2B; no longer U6.S2B
- net MCU_SPI_MISO: now also U4.S1B; no longer U1.S1B
- net MCU_SPI_MOSI: now also U7.S1B; no longer U6.S1B
- net MCU_SWDCLK/TCK: now also J2.SWDCLK/TCK; no longer J5.SWDCLK/TCK
- net MCU_SWDIO/TMS: now also J2.SWDIO/TMS; no longer J5.SWDIO/TMS
- net MCU_SWO/TDO: now also J2.SWO/TDO; no longer J5.SWO/TDO
- net MUX_MCU2USB: now also Q2.C, R11.1, U4.IN, U7.IN; no longer Q1.C, R18.1, U1.IN, U6.IN
- net N$1: now also C6.2, C7.2, L1.1, U2.DVDD; no longer C26.2, C27.2, L3.1, U4.DVDD
- net N$10: now also R12.1; no longer R10.1
- net N$11: now also C17.1, L2.1; no longer C11.1, L1.1
- net N$12: now also C12.1; no longer C5.1
- net N$13: now also C13.1; no longer C6.1
- net N$14: now also Q2.B, R10.1; no longer Q1.B, R19.1
- net N$15: now also C14.1; no longer C7.1
- net N$16: now also C10.2, U2.PMOS; no longer C28.2, U4.PMOS
- net N$17: now also C15.2, U2.!RESET; no longer C29.2, U4.!RESET
- net N$18: now also R6.1, U2.RREF; no longer R22.1, U4.RREF
- net N$19: now also L1.2, U2.AVDD; no longer L3.2, U4.AVDD
- net N$2: now also C2.1, C5.1, U1.+IN; no longer C20.1, C22.1, U5.+IN
- net N$20: now also R17.1, R18.2; no longer R21.1, R24.2
- net N$21: now also U2.USB_N, X1.2; no longer U4.USB_N, X2.2
- net N$22: now also U2.USB_P, X1.3; no longer U4.USB_P, X2.3
- net N$23: now also R5.1, U2.LED; no longer R23.1, U4.LED
- net N$24: now also R5.2; no longer R23.2
- net N$25: now also C27.2, R18.1, R19.2, U6.IN-; no longer C2.2, R24.1, R25.2, U7.IN-
- net N$3: now also R14.1, R15.2; no longer R4.1, R5.2
- net N$4: now also U1.-IN, U1.OUT; no longer U5.-IN, U5.OUT
- net N$5: now also C21.2, R15.1, R16.2, U5.IN-; no longer C1.2, R5.1, R6.2, U2.IN-
- net N$6: now also R13.2, U5.IN+; no longer R7.2, U2.IN+
- net N$7: now also R12.2, R13.1, R7.2, X2-1.KL; no longer R10.2, R7.1, R9.2, X1-1.KL
- net N$8: now also C11.1; no longer C18.1
- net N$9: now also Q1.D, R8.1; no longer Q2.D, R9.1
- net RANGE_UA: now also Q1.G; no longer Q2.G
- net SDCARD_CARD_DETECT: now also CN2.9, R25.1, U2.!SD_CD; no longer CN1.9, R15.1, U4.!SD_CD
- net SDCARD_CLK: now also CN2.5, U7.D2; no longer CN1.5, U6.D2
- net SDCARD_CMD/MOSI: now also CN2.3, R21.1, U7.D1; no longer CN1.3, R13.1, U6.D1
- net SDCARD_DAT0/MISO: now also CN2.7, R23.1, U4.D1; no longer CN1.7, R14.1, U1.D1
- net SDCARD_DAT1: now also CN2.8, U4.D2; no longer CN1.8, U1.D2
- net SDCARD_DAT2: now also CN2.1, U4.D3; no longer CN1.1, U1.D3
- net SDCARD_DAT3/!CS!: now also CN2.2, U4.D4; no longer CN1.2, U1.D4
- net USB_CLK: now also U2.SD_CLK, U7.S2A; no longer U4.SD_CLK, U6.S2A
- net USB_CMD: now also U2.SD_CMD, U7.S1A; no longer U4.SD_CMD, U6.S1A
- net USB_DAT0: now also U2.SD_D0, U4.S1A; no longer U1.S1A, U4.SD_D0
- net USB_DAT1: now also U2.SD_D1, U4.S2A; no longer U1.S2A, U4.SD_D1
- net USB_DAT2: now also U2.SD_D2, U4.S3A; no longer U1.S3A, U4.SD_D2
- net USB_DAT3: now also U2.SD_D3, U4.S4A; no longer U1.S4A, U4.SD_D3
- net USB_VDD: now also C3.2, R10.2, R9.1, U2.VBUS, X1.1; no longer C32.2, R19.2, R20.1, U4.VBUS, X2.1
- net VGND: now also Q1.S, R16.1, R19.1, R4.1, R7.1, X2-2.KL; no longer Q2.S, R12.1, R25.1, R6.1, R8.1, X1-2.KL
Other:
- note added: "1) Reducing the size of the gain-setting resistors and the input-source impedance minimizes the offset error."
- note added: "2) A capacitor in parallel with the feedback resistor reduces the amount of clock feedthrough to the output by limiting the closed-loop bandwidth of the device."
- note added: "2.4 GHz Bluetooth Transceiver Interface"
- note added: "From MAX4238/MAX4239 datasheet:"
- note added: "Full Schematic"
- note added: "Micro SD-Card interface"
- note added: "[MCU or USB] <--> [Micro SD-Card] Communication (MCU as default)"
- note added: "x10"
- note removed: "2.4 GHz Bluetooth Transceiver"
- note removed: "Complete Schematic"
- note removed: "MCU or USB Micro SD-Card Communication (MCU as default)"
- moved on the sheet: C1, C10, C11, C12, C13, C14, C15, C16, C17, C18, C19, C2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

Commit message: MCU pins assignment done
Connections:
- net MCU_I2C_SCL renamed DISPLAY_I2C_SCL
- net MCU_I2C_SDA renamed DISPLAY_I2C_SDA
- net MCU_UART_RX renamed MCU_ICSP_UART_RX
- net MCU_UART_TX renamed MCU_ICSP_UART_TX
- removed net !MCU_SPI_CS!: U4.S4B
- removed net MCU_SPI_CLK: U7.S2B
- removed net MCU_SPI_MISO: U4.S1B
- removed net MCU_SPI_MOSI: U7.S1B
- removed net P02: U3.P0.02/AIN0
- removed net P03: U3.P0.03/AIN1
- removed net P04: U3.P0.04/AIN2
- removed net P05: U3.P0.05/AIN3
- removed net P06: U3.P0.06
- removed net P11: U3.P0.11
- removed net P12: U3.P0.12
- removed net P13: U3.P0.13
- removed net P14: U3.P0.14
- removed net P15: U3.P0.15
- removed net P16: U3.P0.16
- removed net P17: U3.P0.17
- removed net P19: U3.P0.19
- removed net P20: U3.P0.20
- removed net P22: U3.P0.22
- removed net P23: U3.P0.23
- removed net P24: U3.P0.24
- removed net P25: U3.P0.25
- removed net P28: U3.P0.28/AIN4
- removed net P29: U3.P0.29/AIN5
- removed net P30: U3.P0.30/AIN6
- removed net SDCARD_CARD_DETECT: CN2.9, R25.1, U2.!SD_CD
- new net !SDCARD_CARD_DETECT!: CN2.9, R25.1, U2.!SD_CD, U3.P0.24
- new net !SDCARD_SPI_CS!: U3.P0.14, U4.S4B
- new net SDCARD_SPI_CLK: U3.P0.13, U7.S2B
- new net SDCARD_SPI_MISO: U3.P0.11, U4.S1B
- new net SDCARD_SPI_MOSI: U3.P0.12, U7.S1B
- net MCU_ADC_AMMETER_VOUT: now also U3.P0.03/AIN1
- net MCU_ADC_VGND: now also U3.P0.02/AIN0
- net RANGE_MA: now also U3.P0.23
- net RANGE_UA: now also U3.P0.22
Other:
- note added: "From nRF52832 Product Specification v1.4"
- note added: "Recommended usage for low drive, low frequency I/O only."
- moved on the sheet: C1, C11, C12, C13, C14, C4, C8, J1, U3
